Commit message: 1.添加了工具标定的信息; 2.添加了GripperServer作为服务节点，内部控制robotiq，对外提供服务接口

File: motoman/motoman_ma2010_support/urdf/ma2010_with_robotiq140.xacro (robot description, xacro)
@@ -19,5 +19,5 @@
     <parent link="tool0"/>
 	<child link="grasping_frame"/>
-	<origin xyz=" 0.23 0.0 0.0" rpy="0.0 0.0 0.0" />
+	<origin xyz="0.260522 0.0 0.0" rpy="-0.006 0.008 -0.032" />
   </joint>
 </robot>

Commit message: 1.在机械臂模型中粗略集成d435i相机的模型（仅为可视化）；2.coordinator中新增AutoGrasping.srv用来后续服务；3.更新readme

File: motoman/motoman_ma2010_support/urdf/ma2010_with_robotiq140.xacro (robot description, xacro)
@@ -21,3 +21,9 @@
 	<origin xyz="0.260522 0.0 0.0" rpy="-0.006 0.008 -0.032" />
   </joint>
+  <!-- camera -->
+  <xacro:include filename="$(find realsense2_description)/urdf/_d435i.urdf.xacro"/>
+  <xacro:arg name="use_nominal_extrinsics" default="True" />
+  <sensor_d435 parent="grasping_frame">
+    <origin xyz="-0.24435441521426188 0.03398190911800965 0.1142620117698149" rpy="0 0 0"/>
+  </sensor_d435>
 </robot>
